File: pcb/programmer/programmer.kicad_pcb (KiCad board)
At the start: 2 copper layers, 50 x 50 mm, 28 parts, among them J1 USB_C_Receptacle_USB2.0, J2 Pogo pins, J3 power select, Q1 MMBT3904, Q2 MMBT3904, U1 AMS1117-3.3, U2 CH340G, Y1 12MHz

Commit message: gergers generated
Other:
- board text added: "JLCJLCJLCJLC"
Changed lines of the file:
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@@
   (general
     (thickness 1.6)
-    (drawings 28)
+    (drawings 29)
     (tracks 202)
     (zones 0)
@@
     (46 B.CrtYd user)
     (47 F.CrtYd user)
-    (48 B.Fab user hide)
-    (49 F.Fab user hide)
+    (48 B.Fab user)
+    (49 F.Fab user)
   )
   (setup
@@
     (visible_elements 7FFFFFFF)
     (pcbplotparams
-      (layerselection 0x00030_7ffffffe)
+      (layerselection 0x010ff_ffffffff)
       (usegerberextensions false)
       (usegerberattributes true)
@@
       (plotinvisibletext false)
       (padsonsilk false)
-      (subtractmaskfromsilk false)
-      (outputformat 3)
+      (subtractmaskfromsilk true)
+      (outputformat 1)
       (mirror false)
       (drillshape 0)
       (scaleselection 1)
-      (outputdirectory "export/"))
+      (outputdirectory "export/gerber"))
   )
   (net 0 "")
@@
       (effects (font (size 1 1) (thickness 0.15)))
     )
-    (fp_arc (start 7.62 0) (end 7.62 1.778) (angle -180) (layer F.SilkS) (width 0.12))
-    (fp_arc (start 7.62 0) (end 7.62 1.778) (angle -180) (layer F.CrtYd) (width 0.12))
-    (fp_arc (start -7.874 0) (end -7.874 -1.778) (angle -180) (layer F.CrtYd) (width 0.12))
     (fp_line (start 7.62 -1.778) (end -7.874 -1.778) (layer F.CrtYd) (width 0.12))
     (fp_line (start -7.874 1.778) (end 7.62 1.778) (layer F.CrtYd) (width 0.12))
     (fp_line (start 7.62 1.778) (end -8.001 1.778) (layer F.SilkS) (width 0.12))
     (fp_line (start 7.62 -1.778) (end -8.001 -1.778) (layer F.SilkS) (width 0.12))
+    (fp_arc (start 7.62 0) (end 7.62 1.778) (angle -180) (layer F.SilkS) (width 0.12))
+    (fp_arc (start 7.62 0) (end 7.62 1.778) (angle -180) (layer F.CrtYd) (width 0.12))
+    (fp_arc (start -7.874 0) (end -7.874 -1.778) (angle -180) (layer F.CrtYd) (width 0.12))
     (pad 7 thru_hole oval (at 7.62 0 270) (size 1.7 3) (drill 1.1) (layers *.Cu *.Mask)
       (net 9 /RST))
@@
       (effects (font (size 0.5 0.5) (thickness 0.08)))
     )
-    (pad 2 smd roundrect (at 0.9125 0 180) (size 1.025 1.4) (layers F.Cu F.Paste F.Mask) (roundrect_rratio 0.243902)
+    (pad 2 smd roundrect (at 0.9125 0 180) (size 1.025 1.4) (layers F.Cu F.Paste F.Mask) (roundrect_rratio 0.2439004878048781)
       (net 26 "Net-(J1-PadB5)"))
-    (pad 1 smd roundrect (at -0.9125 0 180) (size 1.025 1.4) (layers F.Cu F.Paste F.Mask) (roundrect_rratio 0.243902)
+    (pad 1 smd roundrect (at -0.9125 0 180) (size 1.025 1.4) (layers F.Cu F.Paste F.Mask) (roundrect_rratio 0.2439004878048781)
       (net 1 GND))
     (model ${KISYS3DMOD}/Resistor_SMD.3dshapes/R_0805_2012Metric.wrl
@@
       (effects (font (size 0.5 0.5) (thickness 0.08)))
     )
-    (pad 2 smd roundrect (at 0.9125 0 180) (size 1.025 1.4) (layers F.Cu F.Paste F.Mask) (roundrect_rratio 0.243902)
+    (pad 2 smd roundrect (at 0.9125 0 180) (size 1.025 1.4) (layers F.Cu F.Paste F.Mask) (roundrect_rratio 0.2439004878048781)
       (net 24 "Net-(J1-PadA5)"))
-    (pad 1 smd roundrect (at -0.9125 0 180) (size 1.025 1.4) (layers F.Cu F.Paste F.Mask) (roundrect_rratio 0.243902)
+    (pad 1 smd roundrect (at -0.9125 0 180) (size 1.025 1.4) (layers F.Cu F.Paste F.Mask) (roundrect_rratio 0.2439004878048781)
       (net 1 GND))
     (model ${KISYS3DMOD}/Resistor_SMD.3dshapes/R_0805_2012Metric.wrl
@@
       (effects (font (size 0.5 0.5) (thickness 0.08)))
     )
-    (pad 1 smd roundrect (at -0.9125 0 90) (size 1.025 1.4) (layers F.Cu F.Paste F.Mask) (roundrect_rratio 0.243902)
+    (pad 1 smd roundrect (at -0.9125 0 90) (size 1.025 1.4) (layers F.Cu F.Paste F.Mask) (roundrect_rratio 0.2439004878048781)
       (net 16 "Net-(Q2-Pad1)"))
-    (pad 2 smd roundrect (at 0.9125 0 90) (size 1.025 1.4) (layers F.Cu F.Paste F.Mask) (roundrect_rratio 0.243902)
+    (pad 2 smd roundrect (at 0.9125 0 90) (size 1.025 1.4) (layers F.Cu F.Paste F.Mask) (roundrect_rratio 0.2439004878048781)
       (net 13 /RTS))
     (model ${KISYS3DMOD}/Resistor_SMD.3dshapes/R_0805_2012Metric.wrl
@@
       (effects (font (size 0.5 0.5) (thickness 0.08)))
     )
-    (pad 1 smd roundrect (at -0.9125 0 270) (size 1.025 1.4) (layers F.Cu F.Paste F.Mask) (roundrect_rratio 0.243902)
+    (pad 1 smd roundrect (at -0.9125 0 270) (size 1.025 1.4) (layers F.Cu F.Paste F.Mask) (roundrect_rratio 0.2439004878048781)
       (net 14 "Net-(Q1-Pad1)"))
-    (pad 2 smd roundrect (at 0.9125 0 270) (size 1.025 1.4) (layers F.Cu F.Paste F.Mask) (roundrect_rratio 0.243902)
+    (pad 2 smd roundrect (at 0.9125 0 270) (size 1.025 1.4) (layers F.Cu F.Paste F.Mask) (roundrect_rratio 0.2439004878048781)
       (net 15 /DTR))
     (model ${KISYS3DMOD}/Resistor_SMD.3dshapes/R_0805_2012Metric.wrl
@@
       (effects (font (size 0.5 0.5) (thickness 0.08)))
     )
-    (pad 2 smd roundrect (at 0.9125 0 180) (size 1.025 1.4) (layers F.Cu F.Paste F.Mask) (roundrect_rratio 0.243902)
+    (pad 2 smd roundrect (at 0.9125 0 180) (size 1.025 1.4) (layers F.Cu F.Paste F.Mask) (roundrect_rratio 0.2439004878048781)
       (net 17 "Net-(R2-Pad2)"))
-    (pad 1 smd roundrect (at -0.9125 0 180) (size 1.025 1.4) (layers F.Cu F.Paste F.Mask) (roundrect_rratio 0.243902)
+    (pad 1 smd roundrect (at -0.9125 0 180) (size 1.025 1.4) (layers F.Cu F.Paste F.Mask) (roundrect_rratio 0.2439004878048781)
       (net 12 /TX))
     (model ${KISYS3DMOD}/Resistor_SMD.3dshapes/R_0805_2012Metric.wrl
@@
       (effects (font (size 0.5 0.5) (thickness 0.08)))
     )
-    (pad 2 smd roundrect (at 0.9125 0 180) (size 1.025 1.4) (layers F.Cu F.Paste F.Mask) (roundrect_rratio 0.243902)
+    (pad 2 smd roundrect (at 0.9125 0 180) (size 1.025 1.4) (layers F.Cu F.Paste F.Mask) (roundrect_rratio 0.2439004878048781)
       (net 2 +5V))
-    (pad 1 smd roundrect (at -0.9125 0 180) (size 1.025 1.4) (layers F.Cu F.Paste F.Mask) (roundrect_rratio 0.243902)
+    (pad 1 smd roundrect (at -0.9125 0 180) (size 1.025 1.4) (layers F.Cu F.Paste F.Mask) (roundrect_rratio 0.2439004878048781)
       (net 6 "Net-(D1-Pad2)"))
     (model ${KISYS3DMOD}/Resistor_SMD.3dshapes/R_0805_2012Metric.wrl
@@
       (effects (font (size 0.8 0.8) (thickness 0.12)))
     )
-    (pad 2 smd roundrect (at 1.35 0 90) (size 1.4 1.35) (layers F.Cu F.Paste F.Mask) (roundrect_rratio 0.185185)
+    (pad 2 smd roundrect (at 1.35 0 90) (size 1.4 1.35) (layers F.Cu F.Paste F.Mask) (roundrect_rratio 0.1851844444444445)
       (net 1 GND))
-    (pad 1 smd roundrect (at -1.35 0 90) (size 1.4 1.35) (layers F.Cu F.Paste F.Mask) (roundrect_rratio 0.185185)
+    (pad 1 smd roundrect (at -1.35 0 90) (size 1.4 1.35) (layers F.Cu F.Paste F.Mask) (roundrect_rratio 0.1851844444444445)
       (net 3 +3V3))
     (model ${KISYS3DMOD}/Capacitor_Tantalum_SMD.3dshapes/CP_EIA-3216-10_Kemet-I.wrl
@@
     )
   )
+  (gr_text JLCJLCJLCJLC (at 51.9964 71.9228) (layer F.SilkS)
+    (effects (font (size 0.9 0.9) (thickness 0.15)))
+  )
   (gr_line (start 56.4 45.3) (end 60 45.3) (layer F.SilkS) (width 0.12))
