File: pcb/star/star.sch (KiCad schematic (older format))
At the start: 34 parts, among them J1 POWER, J2 Conn_01x06_Male, SW1 RST, SW2 PRG, U1 ESP-12F, U2 AP2112K-3.3

Commit message: programmer and cad added
Parts:
- removed J2: Conn_01x06_Male, symbol Connector:Conn_01x06_Male
- added J2: program, star:conn_01x07_SMD, symbol Connector:Conn_01x07_Male
Connections:
- net +3V3: now also J2.2 (Pin_2)
- net +5V: now also J2.1 (Pin_1)
- net GND: now also J2.5 (Pin_5)
- net GPIO0: now also J2.6 (Pin_6)
- net RST: now also J2.7 (Pin_7)
- net RXD: now also J2.4 (Pin_4)
- net TXD: now also J2.3 (Pin_3)
Changed lines of the file:
@@
 encoding utf-8
 Sheet 1 1
-Title "Star"
+Title "Christmas star"
 Date "2021-09-02"
 Rev "1"
-Comp "Klushok - B. den Ouden"
-Comment1 ""
-Comment2 "which are sure to create a festive feeling!"
-Comment3 "This christmas star contains 20 individually adressable LEDs"
-Comment4 "A star is born!"
+Comp ""
+Comment1 "B. den Ouden"
+Comment2 ""
+Comment3 ""
+Comment4 ""
 $EndDescr
 $Comp
@@
 L power:+3.3V #PWR0154
 U 1 1 615A1B6A
-P 10550 5100
-F 0 "#PWR0154" H 10550 4950 50  0001 C CNN
-F 1 "+3.3V" H 10565 5273 50  0000 C CNN
-F 2 "" H 10550 5100 50  0001 C CNN
-F 3 "" H 10550 5100 50  0001 C CNN
-	1    10550 5100
-	1    0    0    -1
-$EndComp
-Wire Wire Line
-	10100 5150 10550 5150
-Wire Wire Line
-	10550 5150 10550 5100
+P 10700 4900
+F 0 "#PWR0154" H 10700 4750 50  0001 C CNN
+F 1 "+3.3V" H 10715 5073 50  0000 C CNN
+F 2 "" H 10700 4900 50  0001 C CNN
+F 3 "" H 10700 4900 50  0001 C CNN
+	1    10700 4900
+	1    0    0    -1
+$EndComp
+Wire Wire Line
+	10100 5150 10700 5150
+Wire Wire Line
+	10700 5150 10700 4900
 Wire Wire Line
 	10100 5250 10300 5250
@@
 Text Label 2000 1100 0    50   ~ 0
 LED_Din
-$Comp
-L Connector:Conn_01x06_Male J2
-U 1 1 615A02DC
-P 9900 5350
-F 0 "J2" H 10008 5731 50  0000 C CNN
-F 1 "Conn_01x06_Male" H 10008 5640 50  0000 C CNN
-F 2 "" H 9900 5350 50  0001 C CNN
-F 3 "~" H 9900 5350 50  0001 C CNN
-	1    9900 5350
-	1    0    0    -1
-$EndComp
 Wire Wire Line
 	2000 1100 1550 1100
@@
 NoConn ~ 7700 3300
 NoConn ~ 7800 3300
+$Comp
+L Connector:Conn_01x07_Male J2
+U 1 1 613D463C
+P 9900 5350
+F 0 "J2" H 10008 5831 50  0000 C CNN
+F 1 "program" H 10008 5740 50  0000 C CNN
+F 2 "star:conn_01x07_SMD" H 9900 5350 50  0001 C CNN
+F 3 "~" H 9900 5350 50  0001 C CNN
+	1    9900 5350
+	1    0    0    -1
+$EndComp
+$Comp
+L power:+5V #PWR0156
+U 1 1 613E0FF3
+P 10400 4900
+F 0 "#PWR0156" H 10400 4750 50  0001 C CNN
+F 1 "+5V" H 10415 5073 50  0000 C CNN
+F 2 "" H 10400 4900 50  0001 C CNN
+F 3 "" H 10400 4900 50  0001 C CNN
+	1    10400 4900
+	1    0    0    -1
+$EndComp
+Wire Wire Line
+	10100 5050 10400 5050
+Wire Wire Line
+	10400 5050 10400 4900
 $EndSCHEMATC

Commit message: led pin changed to GPIO2
Connections:
- net LED_Din: now also D16.4 (DI), U1.11 (GPIO2); no longer D20.4 (DI), U1.14 (GPIO5)
- net DoD20: now reaches D1.4 (DI), D20.1 (DO)
- net at D19.1 (DO): now also D20.4 (DI)
- net DoD15: no longer names the net of D15.1 (DO)
- net DoD15: no longer D16.4 (DI)
- no-connect marks 14 -> 15
Other:
- moved on the sheet: D16, D17, D18, D19, D20
Changed lines of the file:
@@
 L LED:APA-106-F5 D16
 U 1 1 61337BDE
-P 4950 2300
-F 0 "D16" H 5294 2346 50  0000 L CNN
-F 1 "APA-106-F5" H 5294 2255 50  0000 L CNN
-F 2 "LED_THT:LED_D5.0mm-4_RGB" H 5000 2000 50  0001 L TNN
-F 3 "https://cdn.sparkfun.com/datasheets/Components/LED/COM-12877.pdf" H 5050 1925 50  0001 L TNN
-	1    4950 2300
+P 5000 2300
+F 0 "D16" H 5344 2346 50  0000 L CNN
+F 1 "APA-106-F5" H 5344 2255 50  0000 L CNN
+F 2 "LED_THT:LED_D5.0mm-4_RGB" H 5050 2000 50  0001 L TNN
+F 3 "https://cdn.sparkfun.com/datasheets/Components/LED/COM-12877.pdf" H 5100 1925 50  0001 L TNN
+	1    5000 2300
 	1    0    0    -1
 $EndComp
@@
 L LED:APA-106-F5 D17
 U 1 1 61337BE4
-P 4950 3400
-F 0 "D17" H 4606 3446 50  0000 R CNN
-F 1 "APA-106-F5" H 4606 3355 50  0000 R CNN
-F 2 "LED_THT:LED_D5.0mm-4_RGB" H 5000 3100 50  0001 L TNN
-F 3 "https://cdn.sparkfun.com/datasheets/Components/LED/COM-12877.pdf" H 5050 3025 50  0001 L TNN
-	1    4950 3400
+P 5000 3400
+F 0 "D17" H 4656 3446 50  0000 R CNN
+F 1 "APA-106-F5" H 4656 3355 50  0000 R CNN
+F 2 "LED_THT:LED_D5.0mm-4_RGB" H 5050 3100 50  0001 L TNN
+F 3 "https://cdn.sparkfun.com/datasheets/Components/LED/COM-12877.pdf" H 5100 3025 50  0001 L TNN
+	1    5000 3400
 	-1   0    0    -1
 $EndComp
@@
 L LED:APA-106-F5 D18
 U 1 1 61337BEA
-P 4950 4500
-F 0 "D18" H 5294 4546 50  0000 L CNN
-F 1 "APA-106-F5" H 5294 4455 50  0000 L CNN
-F 2 "LED_THT:LED_D5.0mm-4_RGB" H 5000 4200 50  0001 L TNN
-F 3 "https://cdn.sparkfun.com/datasheets/Components/LED/COM-12877.pdf" H 5050 4125 50  0001 L TNN
-	1    4950 4500
+P 5000 4500
+F 0 "D18" H 5344 4546 50  0000 L CNN
+F 1 "APA-106-F5" H 5344 4455 50  0000 L CNN
+F 2 "LED_THT:LED_D5.0mm-4_RGB" H 5050 4200 50  0001 L TNN
+F 3 "https://cdn.sparkfun.com/datasheets/Components/LED/COM-12877.pdf" H 5100 4125 50  0001 L TNN
+	1    5000 4500
 	1    0    0    -1
 $EndComp
@@
 L LED:APA-106-F5 D19
 U 1 1 61337BF0
-P 4950 5600
-F 0 "D19" H 4606 5646 50  0000 R CNN
-F 1 "APA-106-F5" H 4606 5555 50  0000 R CNN
-F 2 "LED_THT:LED_D5.0mm-4_RGB" H 5000 5300 50  0001 L TNN
-F 3 "https://cdn.sparkfun.com/datasheets/Components/LED/COM-12877.pdf" H 5050 5225 50  0001 L TNN
-	1    4950 5600
+P 5000 5600
+F 0 "D19" H 4656 5646 50  0000 R CNN
+F 1 "APA-106-F5" H 4656 5555 50  0000 R CNN
+F 2 "LED_THT:LED_D5.0mm-4_RGB" H 5050 5300 50  0001 L TNN
+F 3 "https://cdn.sparkfun.com/datasheets/Components/LED/COM-12877.pdf" H 5100 5225 50  0001 L TNN
+	1    5000 5600
 	-1   0    0    -1
 $EndComp
@@
 L power:+5V #PWR0104
 U 1 1 613672DC
-P 4950 2000
-F 0 "#PWR0104" H 4950 1850 50  0001 C CNN
-F 1 "+5V" H 4965 2173 50  0000 C CNN
-F 2 "" H 4950 2000 50  0001 C CNN
-F 3 "" H 4950 2000 50  0001 C CNN
-	1    4950 2000
+P 5000 2000
+F 0 "#PWR0104" H 5000 1850 50  0001 C CNN
+F 1 "+5V" H 5015 2173 50  0000 C CNN
+F 2 "" H 5000 2000 50  0001 C CNN
+F 3 "" H 5000 2000 50  0001 C CNN
+	1    5000 2000
 	1    0    0    -1
 $EndComp
@@
 L power:GND #PWR0105
 U 1 1 61367CCB
-P 4950 2600
-F 0 "#PWR0105" H 4950 2350 50  0001 C CNN
-F 1 "GND" H 4955 2427 50  0000 C CNN
-F 2 "" H 4950 2600 50  0001 C CNN
-F 3 "" H 4950 2600 50  0001 C CNN
-	1    4950 2600
+P 5000 2600
+F 0 "#PWR0105" H 5000 2350 50  0001 C CNN
+F 1 "GND" H 5005 2427 50  0000 C CNN
+F 2 "" H 5000 2600 50  0001 C CNN
+F 3 "" H 5000 2600 50  0001 C CNN
+	1    5000 2600
 	1    0    0    -1
 $EndComp
@@
 L power:+5V #PWR0106
 U 1 1 613743C2
-P 4950 3100
-F 0 "#PWR0106" H 4950 2950 50  0001 C CNN
-F 1 "+5V" H 4965 3273 50  0000 C CNN
-F 2 "" H 4950 3100 50  0001 C CNN
-F 3 "" H 4950 3100 50  0001 C CNN
-	1    4950 3100
+P 5000 3100
+F 0 "#PWR0106" H 5000 2950 50  0001 C CNN
+F 1 "+5V" H 5015 3273 50  0000 C CNN
+F 2 "" H 5000 3100 50  0001 C CNN
+F 3 "" H 5000 3100 50  0001 C CNN
+	1    5000 3100
 	1    0    0    -1
 $EndComp
@@
 L power:GND #PWR0107
 U 1 1 613743C8
-P 4950 3700
-F 0 "#PWR0107" H 4950 3450 50  0001 C CNN
-F 1 "GND" H 4955 3527 50  0000 C CNN
-F 2 "" H 4950 3700 50  0001 C CNN
-F 3 "" H 4950 3700 50  0001 C CNN
-	1    4950 3700
+P 5000 3700
+F 0 "#PWR0107" H 5000 3450 50  0001 C CNN
+F 1 "GND" H 5005 3527 50  0000 C CNN
+F 2 "" H 5000 3700 50  0001 C CNN
+F 3 "" H 5000 3700 50  0001 C CNN
+	1    5000 3700
 	1    0    0    -1
 $EndComp
@@
 L power:+5V #PWR0108
 U 1 1 61375356
-P 4950 4200
-F 0 "#PWR0108" H 4950 4050 50  0001 C CNN
-F 1 "+5V" H 4965 4373 50  0000 C CNN
-F 2 "" H 4950 4200 50  0001 C CNN
-F 3 "" H 4950 4200 50  0001 C CNN
-	1    4950 4200
+P 5000 4200
+F 0 "#PWR0108" H 5000 4050 50  0001 C CNN
+F 1 "+5V" H 5015 4373 50  0000 C CNN
+F 2 "" H 5000 4200 50  0001 C CNN
+F 3 "" H 5000 4200 50  0001 C CNN
+	1    5000 4200
 	1    0    0    -1
 $EndComp
@@
 L power:GND #PWR0109
 U 1 1 6137535C
-P 4950 4800
-F 0 "#PWR0109" H 4950 4550 50  0001 C CNN
-F 1 "GND" H 4955 4627 50  0000 C CNN
-F 2 "" H 4950 4800 50  0001 C CNN
-F 3 "" H 4950 4800 50  0001 C CNN
-	1    4950 4800
+P 5000 4800
+F 0 "#PWR0109" H 5000 4550 50  0001 C CNN
+F 1 "GND" H 5005 4627 50  0000 C CNN
+F 2 "" H 5000 4800 50  0001 C CNN
+F 3 "" H 5000 4800 50  0001 C CNN
+	1    5000 4800
 	1    0    0    -1
 $EndComp
@@
 L power:+5V #PWR0110
 U 1 1 61376404
-P 4950 5300
-F 0 "#PWR0110" H 4950 5150 50  0001 C CNN
-F 1 "+5V" H 4965 5473 50  0000 C CNN
-F 2 "" H 4950 5300 50  0001 C CNN
-F 3 "" H 4950 5300 50  0001 C CNN
-	1    4950 5300
+P 5000 5300
+F 0 "#PWR0110" H 5000 5150 50  0001 C CNN
+F 1 "+5V" H 5015 5473 50  0000 C CNN
+F 2 "" H 5000 5300 50  0001 C CNN
+F 3 "" H 5000 5300 50  0001 C CNN
+	1    5000 5300
 	1    0    0    -1
 $EndComp
@@
 L power:GND #PWR0111
 U 1 1 6137640A
-P 4950 5900
-F 0 "#PWR0111" H 4950 5650 50  0001 C CNN
-F 1 "GND" H 4955 5727 50  0000 C CNN
-F 2 "" H 4950 5900 50  0001 C CNN
-F 3 "" H 4950 5900 50  0001 C CNN
-	1    4950 5900
+P 5000 5900
+F 0 "#PWR0111" H 5000 5650 50  0001 C CNN
+F 1 "GND" H 5005 5727 50  0000 C CNN
+F 2 "" H 5000 5900 50  0001 C CNN
+F 3 "" H 5000 5900 50  0001 C CNN
+	1    5000 5900
 	1    0    0    -1
 $EndComp
@@
 	4150 4400 4050 4400
 Wire Wire Line
-	5250 4400 5350 4400
-Wire Wire Line
-	5350 4400 5350 5500
-Wire Wire Line
-	5350 5500 5250 5500
+	5300 4400 5400 4400
+Wire Wire Line
+	5400 4400 5400 5500
+Wire Wire Line
+	5400 5500 5300 5500
 Wire Wire Line
 	3450 4400 3350 4400
@@
 	4150 3300 4050 3300
 Wire Wire Line
-	5250 2200 5350 2200
-Wire Wire Line
-	5350 2200 5350 3300
-Wire Wire Line
-	5350 3300 5250 3300
-Wire Wire Line
-	4650 4400 4550 4400
-Wire Wire Line
-	4550 4400 4550 3300
-Wire Wire Line
-	4550 3300 4650 3300
+	5300 2200 5400 2200
+Wire Wire Line
+	5400 2200 5400 3300
+Wire Wire Line
+	5400 3300 5300 3300
+Wire Wire Line
+	4700 4400 4600 4400
+Wire Wire Line
+	4600 4400 4600 3300
+Wire Wire Line
+	4600 3300 4700 3300
 Text Label 1650 6600 0    50   ~ 0
 DoD5
@@
 Wire Wire Line
 	3350 2200 3450 2200
-Text Label 4150 6600 0    50   ~ 0
-DoD15
-Wire Wire Line
-	4150 6600 4050 6600
-Text Label 4550 2200 2    50   ~ 0
-DoD15
-Wire Wire Line
-	4550 2200 4650 2200
+Text Label 5400 6600 0    50   ~ 0
+DoD20
+Text Label 850  2200 2    50   ~ 0
+DoD20
+Wire Wire Line
+	4600 2200 4700 2200
 $Comp
 L power:+3.3V #PWR0144
@@
 Wire Wire Line
 	8650 2800 8450 2800
-Text Label 8550 2300 0    50   ~ 0
+Text Label 8550 2600 0    50   ~ 0
 LED_Din
 Wire Wire Line
-	8550 2300 8450 2300
+	8550 2600 8450 2600
 Text Label 6600 2100 2    50   ~ 0
 RST
@@
 	8000 5750 8000 5650
 $Comp
-L power:GND #PWR0113
-U 1 1 613771D0
-P 1250 1500
-F 0 "#PWR0113" H 1250 1250 50  0001 C CNN
-F 1 "GND" H 1255 1327 50  0000 C CNN
-F 2 "" H 1250 1500 50  0001 C CNN
-F 3 "" H 1250 1500 50  0001 C CNN
-	1    1250 1500
-	1    0    0    -1
-$EndComp
-$Comp
 L power:+5V #PWR0112
 U 1 1 613771CA
-P 1250 900
-F 0 "#PWR0112" H 1250 750 50  0001 C CNN
-F 1 "+5V" H 1265 1073 50  0000 C CNN
-F 2 "" H 1250 900 50  0001 C CNN
-F 3 "" H 1250 900 50  0001 C CNN
-	1    1250 900
+P 5000 6400
+F 0 "#PWR0112" H 5000 6250 50  0001 C CNN
+F 1 "+5V" H 5015 6573 50  0000 C CNN
+F 2 "" H 5000 6400 50  0001 C CNN
+F 3 "" H 5000 6400 50  0001 C CNN
+	1    5000 6400
 	1    0    0    -1
 $EndComp
@@
 L LED:APA-106-F5 D20
 U 1 1 61337BF6
-P 1250 1200
-F 0 "D20" H 906 1246 50  0000 R CNN
-F 1 "APA-106-F5" H 906 1155 50  0000 R CNN
-F 2 "LED_THT:LED_D5.0mm-4_RGB" H 1300 900 50  0001 L TNN
-F 3 "https://cdn.sparkfun.com/datasheets/Components/LED/COM-12877.pdf" H 1350 825 50  0001 L TNN
-	1    1250 1200
-	-1   0    0    -1
-$EndComp
-Text Label 2000 1100 0    50   ~ 0
+P 5000 6700
+F 0 "D20" H 5500 6700 50  0000 R CNN
+F 1 "APA-106-F5" H 5850 6600 50  0000 R CNN
+F 2 "LED_THT:LED_D5.0mm-4_RGB" H 5050 6400 50  0001 L TNN
+F 3 "https://cdn.sparkfun.com/datasheets/Components/LED/COM-12877.pdf" H 5100 6325 50  0001 L TNN
+	1    5000 6700
+	1    0    0    -1
+$EndComp
+Text Label 4600 2200 2    50   ~ 0
 LED_Din
-Wire Wire Line
-	2000 1100 1550 1100
-Wire Wire Line
-	950  1100 850  1100
-Wire Wire Line
-	850  1100 850  2200
 Wire Wire Line
 	850  2200 950  2200
@@
 NoConn ~ 6650 2700
 NoConn ~ 8450 2700
-NoConn ~ 8450 2600
+NoConn ~ 8450 2300
 NoConn ~ 8450 2400
 NoConn ~ 7300 3300
@@
 Wire Wire Line
 	10400 5050 10400 4900
+Wire Wire Line
+	4700 5500 4600 5500
+Wire Wire Line
+	4600 5500 4600 6600
+Wire Wire Line
+	4600 6600 4700 6600
+$Comp
+L power:GND #PWR0113
+U 1 1 614142FA
+P 5000 7000
+F 0 "#PWR0113" H 5000 6750 50  0001 C CNN
+F 1 "GND" H 5005 6827 50  0000 C CNN
+F 2 "" H 5000 7000 50  0001 C CNN
+F 3 "" H 5000 7000 50  0001 C CNN
+	1    5000 7000
+	1    0    0    -1
+$EndComp
+Wire Wire Line
+	5400 6600 5300 6600
+NoConn ~ 4050 6600
 $EndSCHEMATC

Commit message: ibom added
Parts:
- added R4: 10k, Resistor_THT:R_Axial_DIN0204_L3.6mm_D1.6mm_P7.62mm_Horizontal, symbol Device:R
Connections:
- net GND: now also R4.1
- net at U1.10 (GPIO15): now also R4.2
- no-connect marks 15 -> 14
Other:
- note added: "20x apa106 LED"
- note added: "ESP12F microcontroller"
- note added: "Flash button"
- note added: "Power connector and voltage regulator"
- note added: "Programming connectors\n"
- note added: "Reset button"
- moved on the sheet: C1, C2, C3, C4, C5, D1, D10, D11, D12, D13, D14, D15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
